File: hardware/kicad/WPT-TX/WPT-01-TRANSMITTER.kicad_pcb (KiCad board)
At the start: 4 copper layers, 70 x 85 mm, 202 parts, among them CN201 ULO-FH411-1*15SF11, CN202 ULO-FH411-1*15SF11, CN203 ULO-PH409-1*3SF11, CN204 ULO-FH411-1*15SF11, CN205 ULO-FH411-1*15SF11, CN206 SM04B-SRSS-TB(LF)(SN), CN207 ULO-PH409-1*3SF11, CN208 ULO-PH409-1*2SF11, CN209 ULO-PH409-1*2SF11, CN210 ULO-PH409-1*2SF11, CN301 CON-SMA-EDGE-S, CN302 ULO-PH409-1*2SF11, J201 %R, J202 ULO-PH409-1*2SF11, Q301 EPC2038, Q302 EPC2007C, Q303 EPC2007C, Q304 EPC2038, Q305 EPC2007C, Q306 EPC2007C, U201 TS30042-M000QFNR, U202 PCA9306DCUR, U203 PAC1720-1-AIA-TR, U204 MCP45HV51-104E_ST, U205 NCP1117LPST50T3G, U206 MIC5504-3.3YM5-TR, U207 TS30042-M000QFNR, U301 74LVC1G34SE-7, U302 LM5113QDPRRQ1, U303 74LVC1G04SE-7, U304 74LVC1G04SE-7, U305 LM5113QDPRRQ1, U306 SI5351A-B-GTR, U307 74LVC1G34SE-7, X301 FA-238_25.0000MB-K3

Commit message: add basic parts for stm based board
Parts:
- removed CN201, CN202, CN204, CN205: ULO-FH411-1*15SF11, ulo:ULO-FH411-1x15SX1
- removed CN206: SM04B-SRSS-TB(LF)(SN), Connectors_JST:SM04B-SRSS-TB
- removed R203: 0, yageo:R_0603
- removed R204: OPEN, yageo:R_0603
- removed the REF** at (205.0, 205.0)
- removed the REF** at (163.0, 130.0)
- removed the REF** at (189.4, 139.6)
- removed the REF** at (216.8, 196.8)
- removed the REF** at (200.0, 205.0)
- removed the REF** at (163.0, 205.0)
- removed the REF** at (168.0, 205.0)
- removed the REF** at (155.0, 205.0)
- removed the REF** at (215.0, 205.0)
- removed the REF** at (215.0, 130.0)
- removed the REF** at (168.0, 130.0)
- removed the REF** at (155.0, 130.0)
- removed TP201, TP202, TP204, TP205, TP207: TP1.0, TestPoint:TP_1mm
- added C1: 100n, Capacitor_SMD:C_0402_1005Metric, F.Cu at (119.4, 156.4)
- added C10: 100n, Capacitor_SMD:C_0402_1005Metric, F.Cu at (125.2, 158.4)
- added C11: 12p, Capacitor_SMD:C_0402_1005Metric, F.Cu at (125.2, 160.4)
- added C12: 12p, Capacitor_SMD:C_0402_1005Metric, F.Cu at (125.2, 162.3)
- added C2: 100n, Capacitor_SMD:C_0402_1005Metric, F.Cu at (119.4, 158.4)
- added C3: 100n, Capacitor_SMD:C_0402_1005Metric, F.Cu at (119.4, 160.4)
- added C4: 100n, Capacitor_SMD:C_0402_1005Metric, F.Cu at (119.4, 162.3)
- added C5: 4.7u, Capacitor_SMD:C_0402_1005Metric, F.Cu at (122.3, 156.4)
- added C6: 10n, Capacitor_SMD:C_0402_1005Metric, F.Cu at (122.3, 158.4)
- added C7: 1u, Capacitor_SMD:C_0402_1005Metric, F.Cu at (122.3, 160.4)
- added C8: 100n, Capacitor_SMD:C_0402_1005Metric, F.Cu at (122.3, 162.3)
- added C9: 1u, Capacitor_SMD:C_0402_1005Metric, F.Cu at (125.2, 156.4)
- added J1: Conn_01x02_Pin, Connector_PinHeader_2.54mm:PinHeader_1x02_P2.54mm_Vertical, F.Cu at (128.9, 157.7)
- added R1: 0, Resistor_SMD:R_0402_1005Metric, F.Cu at (132.7, 160.1)
- added R2: 10k, Resistor_SMD:R_0402_1005Metric, F.Cu at (132.7, 162.1)
- added U2: STM32G474RETx, Package_QFP:LQFP-64_10x10mm_P0.5mm, F.Cu at (125.2, 148.2)
- added Y1: FA-128 24.0000MF10Z-W3, Crystal:Crystal_SMD_SeikoEpson_FA128-4Pin_2.0x1.6mm, F.Cu at (133.2, 157.3)
- J201: value %R -> 54-00129
Connections:
- J201 pad 3: (no net) -> unconnected-(J201-~-Pad3)
- R213 pad 2: /WPT-01-TRANSMITTER-POWER/HVDCDC_EN -> /MCU/GPIO_HVDCDC_EN
- R223 pad 2: /WPT-01-TRANSMITTER-POWER/~WLAT -> /WPT-01-TRANSMITTER-POWER/~{WLAT}
- U201 pad 6: (no net) -> unconnected-(U201-NC-Pad6)
- U201 pad 7: (no net) -> unconnected-(U201-NC-Pad7)
- U203 pad 7: /WPT-01-TRANSMITTER-POWER/~ALERT -> /WPT-01-TRANSMITTER-POWER/~{ALERT}
- U204 pad 7: (no net) -> unconnected-(U204-NC-Pad7)
- U206 pad 4: (no net) -> unconnected-(U206-NC-Pad4)
- U207 pad 6: (no net) -> unconnected-(U207-NC-Pad6)
- U207 pad 7: (no net) -> unconnected-(U207-NC-Pad7)
- U301 pad 1: (no net) -> unconnected-(U301-NC-Pad1)
- U303 pad 1: (no net) -> unconnected-(U303-NC-Pad1)
- U304 pad 1: (no net) -> unconnected-(U304-NC-Pad1)
- U306 pad 6: (no net) -> unconnected-(U306-CLK2-Pad6)
- U306 pad 9: (no net) -> unconnected-(U306-CLK1-Pad9)
- U307 pad 1: (no net) -> unconnected-(U307-NC-Pad1)
Routing:
- net /WPT-01-TRANSMITTER-POWER/~WLAT: track 76.8 -> 0.00 mm, vias 2 -> 0
- net /WPT-01-TRANSMITTER-POWER/HVDCDC_EN: track 66.8 -> 0.00 mm, vias 1 -> 0
- net /WPT-01-TRANSMITTER-POWER/ADC_VDC: track 42.3 -> 3.98 mm, vias 1 -> 0
- net /WPT-01-TRANSMITTER-POWER/~ALERT: track 33.1 -> 0.00 mm, vias 1 -> 0
- net /WPT-01-TRANSMITTER-POWER/SCL: track 35.6 -> 6.65 mm
- net /WPT-01-TRANSMITTER-POWER/SDA: track 26.7 -> 1.00 mm
- net /WPT-01-TRANSMITTER-POWER/VIN: track 36.6 -> 13.3 mm
- net +3V3: track 67.3 -> 61.0 mm, vias 5 -> 3
- net GND: track 196.2 -> 193.2 mm, vias 159 -> 156
- net Net-(CN204-Pad9): track 3.04 -> 0.00 mm
- net Net-(CN204-Pad6): track 3.04 -> 0.00 mm
- net Net-(CN204-Pad5): track 3.04 -> 0.00 mm
- net Net-(CN204-Pad4): track 3.04 -> 0.00 mm
- net Net-(CN204-Pad3): track 3.04 -> 0.00 mm
- net Net-(CN204-Pad15): track 3.04 -> 0.00 mm
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- removed copper zone on B.Cu, net (none)
- removed copper zone on F.Cu, net (none)
- removed copper zone on In1.Cu, net (none)
- removed copper zone on In2.Cu, net (none)
Other:
- board size 70 x 85 mm -> 70 x 65 mm
- net class Default removed
- board text removed: "JLCJLCJLCJLC"
- board text removed: "V-Cut"
- board text removed: "WPT-Transmitter t = 1.6mm 2020/02/22"
