File: hardware/kicad/WPT-TX/WPT-01-TRANSMITTER.kicad_pcb (KiCad board)
At the start: 4 copper layers, 70 x 65 mm, 195 parts, among them CN203 ULO-PH409-1*3SF11, CN207 ULO-PH409-1*3SF11, CN208 ULO-PH409-1*2SF11, CN209 ULO-PH409-1*2SF11, CN210 ULO-PH409-1*2SF11, CN301 CON-SMA-EDGE-S, CN302 ULO-PH409-1*2SF11, J1 Conn_01x02_Pin, J201 54-00129, J202 ULO-PH409-1*2SF11, Q301 EPC2038, Q302 EPC2007C, Q303 EPC2007C, Q304 EPC2038, Q305 EPC2007C, Q306 EPC2007C, U2 STM32G474RETx, U201 TS30042-M000QFNR, U202 PCA9306DCUR, U203 PAC1720-1-AIA-TR, U204 MCP45HV51-104E_ST, U205 NCP1117LPST50T3G, U206 MIC5504-3.3YM5-TR, U207 TS30042-M000QFNR, U301 74LVC1G34SE-7, U302 LM5113QDPRRQ1, U303 74LVC1G04SE-7, U304 74LVC1G04SE-7, U305 LM5113QDPRRQ1, U306 SI5351A-B-GTR, U307 74LVC1G34SE-7, X301 FA-238_25.0000MB-K3, Y1 FA-128 24.0000MF10Z-W3

Commit message: sch: DISP_DC rename, VDDA PWR_FLAG, import parts to PCB
- rename GPIO_DISP_DDC -> GPIO_DISP_DC (sch, pcb net, ioc)
- add PWR_FLAG on VDDA net (clears ERC power_pin_not_driven)
- fix J301 Conn_01x08_Pin description to match library
- pcb: import new footprints from schematic, parked off-board (no placement)

Co-Authored-By: Claude Fable 5.1 <noreply@anthropic.com>
Parts:
- added C338: 1p, Capacitor_SMD:C_0402_1005Metric, F.Cu at (287.8, 179.6)
- added C339: 1p, Capacitor_SMD:C_0402_1005Metric, F.Cu at (291.6, 179.6)
- added J2: Conn_01x12_Pin, Connector_PinHeader_2.54mm:PinHeader_1x12_P2.54mm_Vertical, F.Cu at (237.8, 141.8)
- added J3: Conn_01x05_Pin, Connector_PinHeader_2.54mm:PinHeader_1x05_P2.54mm_Vertical, F.Cu at (285.2, 141.8)
- added J301: Conn_01x08_Pin, Connector_PinHeader_2.54mm:PinHeader_1x08_P2.54mm_Vertical, F.Cu at (243.4, 141.8)
- added J4: Conn_01x04_Pin, Connector_PinHeader_2.54mm:PinHeader_1x04_P2.54mm_Vertical, F.Cu at (290.8, 141.8)
- added J5: USB4105-GF-A, Connector_USB:USB_C_Receptacle_GCT_USB4105-xx-A_16P_TopMnt_Horizontal, F.Cu at (299.9, 144.8)
- added R10: 5.1k, Resistor_SMD:R_0402_1005Metric, F.Cu at (266.6, 174.0)
- added R11: 0, Resistor_SMD:R_0402_1005Metric, F.Cu at (270.5, 174.0)
- added R320: 0, Resistor_SMD:R_0402_1005Metric, F.Cu at (274.4, 174.0)
- added R321: 47k, Resistor_SMD:R_0402_1005Metric, F.Cu at (278.3, 174.0)
- added R323: 0, Resistor_SMD:R_0402_1005Metric, F.Cu at (282.2, 174.0)
- added R324: 47k, Resistor_SMD:R_0402_1005Metric, F.Cu at (286.1, 174.0)
- added R326: 0, Resistor_SMD:R_0402_1005Metric, F.Cu at (290.0, 174.0)
- added R327: 47k, Resistor_SMD:R_0402_1005Metric, F.Cu at (293.9, 174.0)
- added R329: 0, Resistor_SMD:R_0402_1005Metric, F.Cu at (297.8, 174.0)
- added R330: 47k, Resistor_SMD:R_0402_1005Metric, F.Cu at (301.8, 174.0)
- added R331: 10k, Resistor_SMD:R_0402_1005Metric, F.Cu at (305.7, 174.0)
- added R332: 10k, Resistor_SMD:R_0402_1005Metric, F.Cu at (237.0, 179.7)
- added R333: 10k, Resistor_SMD:R_0402_1005Metric, F.Cu at (240.9, 179.7)
- added R334: 10k, Resistor_SMD:R_0402_1005Metric, F.Cu at (244.8, 179.7)
- added R335: 0, Resistor_SMD:R_0402_1005Metric, F.Cu at (248.7, 179.7)
- added R336: 100k, Resistor_SMD:R_0402_1005Metric, F.Cu at (252.6, 179.7)
- added R337: 0, Resistor_SMD:R_0402_1005Metric, F.Cu at (256.5, 179.7)
- added R338: 100k, Resistor_SMD:R_0402_1005Metric, F.Cu at (260.4, 179.7)
- added R339: 15k, Resistor_SMD:R_0402_1005Metric, F.Cu at (264.3, 179.7)
- added R340: 1k, Resistor_SMD:R_0402_1005Metric, F.Cu at (268.2, 179.7)
- added R341: 15k, Resistor_SMD:R_0402_1005Metric, F.Cu at (272.1, 179.7)
- added R342: 1k, Resistor_SMD:R_0402_1005Metric, F.Cu at (276.1, 179.7)
- added R343: 1k, Resistor_SMD:R_0402_1005Metric, F.Cu at (280.0, 179.7)
- added R344: 1k, Resistor_SMD:R_0402_1005Metric, F.Cu at (283.9, 179.7)
- added R4: 3.3k, Resistor_SMD:R_0402_1005Metric, F.Cu at (243.1, 174.0)
- added R5: 3.3k, Resistor_SMD:R_0402_1005Metric, F.Cu at (247.0, 174.0)
- added R6: 3.3k, Resistor_SMD:R_0402_1005Metric, F.Cu at (250.9, 174.0)
- added R7: 10k, Resistor_SMD:R_0402_1005Metric, F.Cu at (254.8, 174.0)
- added R8: 15k, Resistor_SMD:R_0402_1005Metric, F.Cu at (258.7, 174.0)
- added R9: 5.1k, Resistor_SMD:R_0402_1005Metric, F.Cu at (262.7, 174.0)
- added SW1: EC11E09244AQ, Rotary_Encoder:RotaryEncoder_Alps_EC11E-Switch_Vertical_H20mm, F.Cu at (265.3, 144.6)
- added SW2: EG2219, Button_Switch_THT:SW_E-Switch_EG2219_DPDT_Angled, F.Cu at (250.5, 143.1)
- added U3: USBLC6-2SC6, Package_TO_SOT_SMD:SOT-23-6, F.Cu at (238.1, 175.4)
Connections:
- R213 pad 2: /MCU/GPIO_HVDCDC_EN -> /HV_EN_SW
- U2 pad 10: unconnected-(U2-PC2-Pad10) -> /MCU/ADC2_IN8_EXTERNAL
- U2 pad 13: /MCU/ADC2_IN2_EXTERNAL -> /VSWA_CMP
- U2 pad 17: /MCU/GPIO_DISP_DDC -> /MCU/GPIO_DISP_DC
- U2 pad 24: /MCU/GPIO_HVDCDC_EN -> /HV_EN_MCU
- U2 pad 30: /MCU/HRTIM1_FLT3 -> /HRTIM1_FLT3
- U2 pad 33: /MCU/HRTIM1_FLT4 -> /HRTIM1_FLT4
- U2 pad 34: /MCU/HRTIM1_CHC1 -> /HRTIM1_CHC1
- U2 pad 35: /MCU/HRTIM1_CHC2 -> /HRTIM1_CHC2
- U2 pad 36: /MCU/HRTIM1_CHD1 -> /HRTIM1_CHD1
- U2 pad 37: /MCU/HRTIM1_CHD2 -> /HRTIM1_CHD2
- U2 pad 44: /MCU/GPIO_VUSB_SENSE -> unconnected-(U2-PA10-Pad44)
- U2 pad 45: /MCU/USB_DM -> /USB_DM
- U2 pad 46: /MCU/USB_DP -> /USB_DP
- U2 pad 52: unconnected-(U2-PC10-Pad52) -> /GPIO_VUSB_SENSE
- U2 pad 53: /MCU/HRTIM1_EEV2 -> /HRTIM1_EEV2
- U2 pad 54: /MCU/HRTIM1_EEV1 -> /HRTIM1_EEV1
- U2 pad 57: /MCU/GPIO_SW_MISC2 -> /HV_SW_STATE
- U2 pad 9: unconnected-(U2-PC1-Pad9) -> /VSWB_CMP
