File: hardware/kicad/WPT-TX/MCU.kicad_sch (KiCad schematic)
At the start: 18 parts, among them J1 Conn_01x02_Pin, U2 STM32G474RETx, Y1 FA-128 24.0000MF10Z-W3

Commit message: VBUS detect pin change
Connections:
- net GPIO_VUSB_SENSE: now also U2.52 (PC10); no longer U2.44 (PA10)
Changed lines of the file:
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@@
 		(at 165.1 132.08)
 	)
-	(no_connect
-		(at 129.54 119.38)
+	(wire
+		(pts
+			(xy 121.92 119.38) (xy 129.54 119.38)
+		)
+		(stroke
+			(width 0)
+			(type default)
+		)
 	)
 	(no_connect
@@
 		)
 	)
-	(wire
-		(pts
-			(xy 165.1 96.52) (xy 172.72 96.52)
-		)
-		(stroke
-			(width 0)
-			(type default)
-		)
+	(no_connect
+		(at 165.1 96.52)
 	)
 	(wire
@@
 	(hierarchical_label "GPIO_VUSB_SENSE"
 		(shape input)
-		(at 172.72 96.52 0)
+		(at 121.92 119.38 180)
 		(effects
 			(font
 				(size 1.27 1.27)
 			)
-			(justify left)
-		)
-	)
+			(justify right)
+		)
+	)

Commit message: HRTIM
Parts:
- removed R3: 0, Resistor_SMD:R_0402_1005Metric, symbol Device:R
Connections:
- net ADC2_IN8_EXTERNAL: now reaches U2.10 (PC2)
- net VSWB_CMP: now reaches U2.9 (PC1)
- net ADC2_IN2_EXTERNAL renamed VSWA_CMP
- no-connect marks 15 -> 13
Changed lines of the file:
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@@
 	)
 	(no_connect
-		(at 129.54 99.06)
-	)
-	(no_connect
 		(at 165.1 129.54)
 	)
@@
 	)
 	(no_connect
-		(at 129.54 96.52)
-	)
-	(no_connect
 		(at 129.54 88.9)
 	)
@@
 		)
 	)
-	(hierarchical_label "ADC2_IN2_EXTERNAL"
+	(hierarchical_label "VSWA_CMP"
 		(shape input)
 		(at 172.72 73.66 0)
@@
 	)
 	(symbol
-		(lib_id "Device:R")
-		(at 4.1911 7.3717 90)
-		(unit 1)
-		(body_style 1)
-		(exclude_from_sim no)
-		(in_bom yes)
-		(on_board yes)
-		(in_pos_files yes)
-		(dnp no)
-		(fields_autoplaced yes)
-		(property "Reference" "R3"
-			(at 4.1911 1.0217 90)
-			(show_name no)
-			(do_not_autoplace no)
-			(effects
-				(font
-					(size 1.27 1.27)
-				)
-			)
-		)
-		(property "Value" "0"
-			(at 4.1911 3.5617 90)
-			(show_name no)
-			(do_not_autoplace no)
-			(effects
-				(font
-					(size 1.27 1.27)
-				)
-			)
-		)
-		(property "Footprint" "Resistor_SMD:R_0402_1005Metric"
-			(at 4.1911 9.1497 90)
-			(hide yes)
-			(show_name no)
-			(do_not_autoplace no)
-			(effects
-				(font
-					(size 1.27 1.27)
-				)
-			)
-		)
-		(property "Datasheet" ""
-			(at 4.1911 7.3717 0)
-			(hide yes)
-			(show_name no)
-			(do_not_autoplace no)
-			(effects
-				(font
-					(size 1.27 1.27)
-				)
-			)
-		)
-		(property "Description" "Resistor"
-			(at 4.1911 7.3717 0)
-			(hide yes)
-			(show_name no)
-			(do_not_autoplace no)
-			(effects
-				(font
-					(size 1.27 1.27)
-				)
-			)
-		)
-		(pin "2"
-		)
-		(pin "1"
-		)
-		(instances
-			(project "WPT-01-TRANSMITTER"
-				(path "/8d93dcf8-c351-4228-94c4-516db1fed557/82df408d-9aab-4d11-a747-ac2cd4d0c268"
-					(reference "R3")
-					(unit 1)
-				)
-			)
-		)
-	)
-	(symbol
 		(lib_id "Device:C")
 		(at 172.72 57.15 0)
@@
 		)
 	)
+	(wire
+		(pts
+			(xy 129.54 96.52) (xy 121.92 96.52)
+		)
+		(stroke
+			(width 0)
+			(type default)
+		)
+	)
+	(hierarchical_label "VSWB_CMP"
+		(shape input)
+		(at 121.92 96.52 180)
+		(effects
+			(font
+				(size 1.27 1.27)
+			)
+			(justify right)
+		)
+	)
+	(wire
+		(pts
+			(xy 129.54 99.06) (xy 121.92 99.06)
+		)
+		(stroke
+			(width 0)
+			(type default)
+		)
+	)
+	(hierarchical_label "ADC2_IN8_EXTERNAL"
+		(shape input)
+		(at 121.92 99.06 180)
+		(effects
+			(font
+				(size 1.27 1.27)
+			)
+			(justify right)
+		)
+	)
