File: hardware/kicad/WPT-TX/MCU.kicad_sch (KiCad schematic)
At the start: 17 parts, among them J1 Conn_01x02_Pin, U2 STM32G474RETx, Y1 FA-128 24.0000MF10Z-W3

Commit message: sch: DISP_DC rename, VDDA PWR_FLAG, import parts to PCB
- rename GPIO_DISP_DDC -> GPIO_DISP_DC (sch, pcb net, ioc)
- add PWR_FLAG on VDDA net (clears ERC power_pin_not_driven)
- fix J301 Conn_01x08_Pin description to match library
- pcb: import new footprints from schematic, parked off-board (no placement)

Co-Authored-By: Claude Fable 5.1 <noreply@anthropic.com>
Connections:
- net GPIO_DISP_DDC renamed GPIO_DISP_DC
Changed lines of the file:
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@@
 		)
 	)
-	(hierarchical_label "GPIO_DISP_DDC"
+	(hierarchical_label "GPIO_DISP_DC"
 		(shape input)
 		(at 172.72 78.74 0)
@@
 		)
 	)
+	(symbol
+		(lib_id "power:PWR_FLAG")
+		(at 167.64 53.34 0)
+		(unit 1)
+		(body_style 1)
+		(exclude_from_sim no)
+		(in_bom yes)
+		(on_board yes)
+		(in_pos_files yes)
+		(dnp no)
+		(property "Reference" "#FLG01"
+			(at 167.64 51.435 0)
+			(hide yes)
+			(show_name no)
+			(do_not_autoplace no)
+			(effects
+				(font
+					(size 1.27 1.27)
+				)
+			)
+		)
+		(property "Value" "PWR_FLAG"
+			(at 167.64 49.1236 0)
+			(show_name no)
+			(do_not_autoplace no)
+			(effects
+				(font
+					(size 1.016 1.016)
+				)
+			)
+		)
+		(property "Footprint" ""
+			(at 167.64 53.34 0)
+			(hide yes)
+			(show_name no)
+			(do_not_autoplace no)
+			(effects
+				(font
+					(size 1.27 1.27)
+				)
+			)
+		)
+		(property "Datasheet" ""
+			(at 167.64 53.34 0)
+			(hide yes)
+			(show_name no)
+			(do_not_autoplace no)
+			(effects
+				(font
+					(size 1.27 1.27)
+				)
+			)
+		)
+		(property "Description" ""
+			(at 167.64 53.34 0)
+			(show_name no)
+			(do_not_autoplace no)
+			(effects
+				(font
+					(size 1.27 1.27)
+				)
+			)
+		)
+		(pin "1"
+		)
+		(instances
+			(project "WPT-01-TRANSMITTER"
+				(path "/8d93dcf8-c351-4228-94c4-516db1fed557/82df408d-9aab-4d11-a747-ac2cd4d0c268"
+					(reference "#FLG01")
+					(unit 1)
+				)
+			)
+		)
+	)
+	(junction
+		(at 167.64 53.34)
+		(diameter 0)
+		(color 0 0 0 0)
+	)
 )
