File: hardware/kicad/WPT-TX/WPT-01-TRANSMITTER-TX.kicad_sch (KiCad schematic)
At the start: 84 parts, among them CN301 CON-SMA-EDGE-S, CN302 ULO-PH409-1*2SF11, Q301 EPC2038, Q302 EPC2007C, Q303 EPC2007C, Q304 EPC2038, Q305 EPC2007C, Q306 EPC2007C, U301 74LVC1G34SE-7, U302 LM5113QDPRRQ1, U303 74LVC1G04SE-7, U304 74LVC1G04SE-7, U305 LM5113QDPRRQ1, U306 SI5351A-B-GTR, U307 74LVC1G34SE-7, X301 FA-238_25.0000MB-K3

Commit message: HRTIM
Parts:
- added C338, C339: 1p, Capacitor_SMD:C_0402_1005Metric, symbol Device:C
- added J301: Conn_01x08_Pin, Connector_PinHeader_2.54mm:PinHeader_1x08_P2.54mm_Vertical, symbol Connector:Conn_01x08_Pin
- added R319, R320, R322, R323, R325, R326, R328, R329, R335, R337: 0, Resistor_SMD:R_0402_1005Metric, symbol Device:R
- added R321, R324, R327, R330: 47k, Resistor_SMD:R_0402_1005Metric, symbol Device:R
- added R331, R332, R333, R334: 10k, Resistor_SMD:R_0402_1005Metric, symbol Device:R
- added R336, R338: 100k, Resistor_SMD:R_0402_1005Metric, symbol Device:R
- added R339, R341: 15k, Resistor_SMD:R_0402_1005Metric, symbol Device:R
- added R340, R342, R343, R344: 1k, Resistor_SMD:R_0402_1005Metric, symbol Device:R
Connections:
- net +3V3: now also R331.1, R333.1
- net GND: now also J301.2 (Pin_2), J301.4 (Pin_4), R321.2, R324.2, R327.2, R330.2, R332.2, R334.2, R336.2, R338.2, R340.2, R342.2
- net H_Sig1: now also R319.2, R320.1, R321.1; no longer D305.2 (A), R305.1
- net H_Sig2: now also R325.2, R326.1, R327.1; no longer D311.2 (A), R315.1
- net L_Sig1: now also R322.2, R323.1, R324.1; no longer D306.2 (A), R307.1
- net L_Sig2: now also R328.2, R329.1, R330.1; no longer D312.2 (A), R318.1
- net OutA: now also C338.1, R339.1
- net OutB: now also C339.1, R341.1
- new net H1_LEG: D305.2 (A), R305.1, R319.1
- new net H2_LEG: D311.2 (A), R315.1, R325.1
- new net HRTIM1_CHC1: R320.2
- new net HRTIM1_CHC2: R323.2
- new net HRTIM1_CHD1: R326.2
- new net HRTIM1_CHD2: R329.2
- new net HRTIM1_EEV1: R335.2, R336.1
- new net HRTIM1_EEV2: R337.2, R338.1
- new net HRTIM1_FLT3: J301.7 (Pin_7), R331.2, R332.1
- new net HRTIM1_FLT4: J301.8 (Pin_8), R333.2, R334.1
- new net L1_LEG: D306.2 (A), R307.1, R322.1
- new net L2_LEG: D312.2 (A), R318.1, R328.1
- new net VSWA_CMP: R343.1
- new net VSWA_SENSE: C338.2, J301.1 (Pin_1), R339.2, R340.1, R343.2
- new net VSWB_CMP: R344.1
- new net VSWB_SENSE: C339.2, J301.3 (Pin_3), R341.2, R342.1, R344.2
- new net ZVS_A_IN: J301.5 (Pin_5), R335.1
- new net ZVS_B_IN: J301.6 (Pin_6), R337.1

Commit message: sch: USB4105, standard headers, drop R_LEG
Parts:
- removed R319, R322, R325, R328: 0, Resistor_SMD:R_0402_1005Metric, symbol Device:R
- D301, D307: footprint SOD-323 -> Diodes_SMD:SOD-323
Connections:
- net H1_LEG is gone; now on net H_Sig1: D305.2 (A), R305.1
- net H2_LEG is gone; now on net H_Sig2: D311.2 (A), R315.1
- net L1_LEG is gone; now on net L_Sig1: D306.2 (A), R307.1
- net L2_LEG is gone; now on net L_Sig2: D312.2 (A), R318.1
