File: hardware/kicad/WPT-TX/WPT-01-TRANSMITTER.kicad_sch (KiCad schematic)
At the start: 15 parts, among them J2 Conn_01x12_Pin, J3 Conn_01x05_Pin, J4 Conn_01x04_Pin, J5 USB4105-GF-A, SW1 EC11E09244AQ, SW2 EG2219, U3 USBLC6-2SC6

Commit message: sch: DISP_DC rename, VDDA PWR_FLAG, import parts to PCB
- rename GPIO_DISP_DDC -> GPIO_DISP_DC (sch, pcb net, ioc)
- add PWR_FLAG on VDDA net (clears ERC power_pin_not_driven)
- fix J301 Conn_01x08_Pin description to match library
- pcb: import new footprints from schematic, parked off-board (no placement)

Co-Authored-By: Claude Fable 5.1 <noreply@anthropic.com>
Connections:
- net MCU/GPIO_DISP_DDC renamed MCU/GPIO_DISP_DC
Other:
- sheet MCU ports: added GPIO_DISP_DC; removed GPIO_DISP_DDC
Changed lines of the file:
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@@
 			)
 		)
-		(pin "GPIO_DISP_DDC" input
+		(pin "GPIO_DISP_DC" input
 			(at 68.58 176.53 180)
 			(effects
